Commit message: PR2/Grey does not exist anymore

File: kurtana_description/parts/kurtana_rack.urdf.xacro (robot description, xacro)
@@ -182,20 +182,20 @@
   <xacro:kurtana_pole_transmission name="kurtana_pitch" />
   <gazebo reference="kurtana_rackplate_link">
-    <material value="PR2/Grey" />
+    <material value="Gazebo/Grey" />
   </gazebo>
   <gazebo reference="kurtana_baseplate_link">
-    <material value="PR2/Grey" />
+    <material value="Gazebo/Grey" />
   </gazebo>
   <gazebo reference="kurtana_pole_link">
-    <material value="PR2/Grey" />
+    <material value="Gazebo/Grey" />
   </gazebo>
   <gazebo reference="kurtana_innerpole_stretch_link">
-    <material value="PR2/Grey" />
+    <material value="Gazebo/Grey" />
   </gazebo>
   <gazebo reference="kurtana_poletop_roll_link">
-    <material value="PR2/Grey" />
+    <material value="Gazebo/Grey" />
   </gazebo>
   <gazebo reference="kurtana_pitchpole_link">
-    <material value="PR2/Grey" />
+    <material value="Gazebo/Grey" />
   </gazebo>
 </robot>
